File: Xbee_Remote_32u4/board/remote_smt.brd (EAGLE design)
At the start: 43.2 x 71.1 mm, 33 parts, among them X1 16MHz, X2 USBPTH

Commit message: Fixed up SMT version, added some files zipped.
Parts:
- added JP2, JP3: FIDUCIAL1.5X3, SparkFun:FIDUCIAL-1.5X3
- C6, C7: value (none) -> 18pF
Connections:
- net 3.3V: no longer U$7.2
Routing:
- net N$7: track 64.6 -> 57.6 mm
- net GND: track 276.5 -> 281.7 mm
- net 3.3V: track 112.6 -> 111.2 mm
Changed lines of the file:
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@@
 <setting verticaltext="up"/>
 </settings>
-<grid distance="0.1" unitdist="inch" unit="inch" style="lines" multiple="1" display="yes" altdistance="0.025" altunitdist="inch" altunit="inch"/>
+<grid distance="0.05" unitdist="inch" unit="inch" style="lines" multiple="1" display="yes" altdistance="0.025" altunitdist="inch" altunit="inch"/>
 <layers>
 <layer number="1" name="Top" color="4" fill="1" visible="yes" active="yes"/>
@@
 <text x="17.145" y="42.545" size="0.508" layer="21" font="vector">.1uF</text>
 <text x="29.845" y="15.24" size="0.508" layer="21" font="vector" rot="R90">10K</text>
-<wire x1="27.305" y1="20.955" x2="27.305" y2="27.94" width="0.2032" layer="41"/>
 <text x="15.24" y="44.45" size="0.762" layer="21" font="vector">4.5V-15V</text>
 <wire x1="12.065" y1="45.72" x2="20.955" y2="45.72" width="0.2032" layer="21"/>
@@
 <wire x1="17.145" y1="40.64" x2="18.415" y2="40.64" width="0.2032" layer="41"/>
 <text x="-25.4" y="73.66" size="10.16" layer="49" font="vector">UNPROVEN DESIGN</text>
+<wire x1="27.305" y1="20.955" x2="27.305" y2="28.575" width="0.4064" layer="41"/>
 </plain>
 <attributes>
@@
 </element>
 <element name="U$1" library="SparkFun" package="7-SEGMENT-1&quot;PTH" value="7-SEGMENT-DISPLAY-1&quot;-RED" x="13.97" y="10.16" rot="R90"/>
-<element name="C6" library="SparkFun" package="0805" value="" x="31.75" y="7.62" rot="R90"/>
-<element name="C7" library="SparkFun" package="0805" value="" x="29.21" y="7.62" rot="R90"/>
+<element name="C6" library="SparkFun" package="0805" value="18pF" x="31.75" y="7.62" smashed="yes" rot="R90">
+<attribute name="NAME" x="30.9245" y="6.858" size="0.4064" layer="25" rot="R90"/>
+<attribute name="VALUE" x="31.369" y="4.953" size="0.4064" layer="27"/>
+</element>
+<element name="C7" library="SparkFun" package="0805" value="18pF" x="29.21" y="7.62" smashed="yes" rot="R90">
+<attribute name="NAME" x="28.3845" y="6.858" size="0.4064" layer="25" rot="R90"/>
+<attribute name="VALUE" x="28.829" y="4.953" size="0.4064" layer="27"/>
+</element>
 <element name="U$11" library="hjohnson_library" package="EG2513-ND" value="SPST_SWITCH" x="36.83" y="64.77"/>
 <element name="U$12" library="hjohnson_library" package="EG2513-ND" value="SPST_SWITCH" x="36.83" y="60.96"/>
@@
 <attribute name="VALUE" x="36.83" y="10.795" size="0.4064" layer="27"/>
 </element>
+<element name="JP2" library="SparkFun" package="FIDUCIAL-1.5X3" value="FIDUCIAL1.5X3" x="1.905" y="69.215"/>
+<element name="JP3" library="SparkFun" package="FIDUCIAL-1.5X3" value="FIDUCIAL1.5X3" x="41.275" y="1.905"/>
 </elements>
 <signals>
@@
 <wire x1="22.225" y1="26.67" x2="22.49" y2="26.67" width="0.4064" layer="1"/>
 <wire x1="10.795" y1="34.025" x2="10.795" y2="33.02" width="0.6096" layer="1"/>
-<wire x1="35" y1="3.81" x2="33.095" y2="1.905" width="0.4064" layer="16"/>
-<wire x1="33.095" y1="1.905" x2="24.005853125" y2="1.905" width="0.4064" layer="16"/>
-<wire x1="24.005853125" y1="1.905" x2="12.7" y2="13.210853125" width="0.4064" layer="16"/>
-<wire x1="12.7" y1="13.210853125" x2="12.7" y2="26.035" width="0.4064" layer="16"/>
 <wire x1="12.7" y1="26.035" x2="13.335" y2="26.67" width="0.4064" layer="16"/>
 <wire x1="13.335" y1="26.67" x2="13.97" y2="26.67" width="0.4064" layer="16"/>
@@
 <vertex x="0" y="71.12"/>
 </polygon>
+<polygon width="0.2032" layer="1" isolate="0.3048" thermals="no">
+<vertex x="28.575" y="36.195"/>
+<vertex x="28.575" y="45.085"/>
+<vertex x="24.765" y="45.085"/>
+<vertex x="23.495" y="43.815"/>
+<vertex x="23.495" y="37.465"/>
+<vertex x="25.4" y="35.56"/>
+<vertex x="28.575" y="35.56"/>
+</polygon>
+<wire x1="35" y1="3.81" x2="35" y2="8.18" width="0.4064" layer="16"/>
+<wire x1="35" y1="8.18" x2="25.4" y2="17.78" width="0.4064" layer="16"/>
+<wire x1="25.4" y1="17.78" x2="13.97" y2="17.78" width="0.4064" layer="16"/>
+<wire x1="13.97" y1="17.78" x2="12.7" y2="19.05" width="0.4064" layer="16"/>
+<wire x1="12.7" y1="19.05" x2="12.7" y2="26.035" width="0.4064" layer="16"/>
+<wire x1="26.67" y1="44.45" x2="26.67" y2="36.83" width="0.4064" layer="16"/>
 </signal>
 <signal name="MOSI">
@@
 <signal name="3.3V">
 <contactref element="XB1" pad="1"/>
-<contactref element="U$7" pad="44"/>
-<contactref element="U$7" pad="24"/>
-<contactref element="U$7" pad="2"/>
 <contactref element="U$7" pad="34"/>
 <contactref element="U$7" pad="14"/>
@@
 <wire x1="38.1" y1="19.685" x2="38.735" y2="20.32" width="0.4064" layer="1"/>
 <wire x1="38.735" y1="20.32" x2="38.735" y2="22.225" width="0.4064" layer="1"/>
-<wire x1="38.735" y1="22.225" x2="37.575" y2="22.225" width="0.4064" layer="1"/>
-<wire x1="37.575" y1="22.225" x2="37.55" y2="22.2" width="0.4064" layer="1"/>
-<wire x1="25.95" y1="28.6" x2="27.75" y2="28.6" width="0.6096" layer="1"/>
-<wire x1="37.55" y1="22.2" x2="36.22" y2="22.2" width="0.4064" layer="1"/>
+<wire x1="38.735" y1="22.225" x2="37.55" y2="22.225" width="0.4064" layer="1"/>
 <wire x1="36.22" y1="22.2" x2="36.195" y2="22.225" width="0.4064" layer="1"/>
 <wire x1="36.195" y1="22.225" x2="36.195" y2="24.13" width="0.4064" layer="1"/>
@@
 <wire x1="35.75" y1="31.2" x2="35.75" y2="28.765" width="0.6096" layer="1"/>
 <wire x1="35.75" y1="28.765" x2="35.56" y2="28.575" width="0.6096" layer="1"/>
-<wire x1="35.56" y1="28.575" x2="27.775" y2="28.575" width="0.6096" layer="1"/>
-<wire x1="27.775" y1="28.575" x2="27.75" y2="28.6" width="0.6096" layer="1"/>
+<wire x1="35.56" y1="28.575" x2="28.791078125" y2="28.575" width="0.4064" layer="1"/>
+<wire x1="28.791078125" y1="28.575" x2="27.75" y2="29.616078125" width="0.4064" layer="1"/>
+<wire x1="27.75" y1="29.616078125" x2="27.75" y2="31.2" width="0.4064" layer="1"/>
 <wire x1="35.56" y1="28.575" x2="35.56" y2="24.765" width="0.6096" layer="1"/>
 <contactref element="C5" pad="A"/>
@@
 <wire x1="24.13" y1="32.38" x2="24.13" y2="30.48" width="0.6096" layer="1"/>
 <wire x1="22.22" y1="34.29" x2="22.22" y2="40.64" width="0.6096" layer="1"/>
-<wire x1="27.75" y1="31.2" x2="27.75" y2="28.6" width="0.6096" layer="1"/>
 <wire x1="22.22" y1="41.905" x2="27.305" y2="46.99" width="0.6096" layer="1"/>
 <wire x1="27.305" y1="46.99" x2="27.305" y2="48.895" width="0.6096" layer="1"/>
 <wire x1="13.97" y1="21.59" x2="15.24" y2="22.86" width="0.4064" layer="16"/>
-<wire x1="25.95" y1="28.6" x2="24.74" y2="28.6" width="0.4064" layer="1"/>
-<wire x1="24.74" y1="28.6" x2="24.13" y2="29.21" width="0.4064" layer="1"/>
-<wire x1="24.13" y1="29.21" x2="24.13" y2="30.48" width="0.4064" layer="1"/>
 <wire x1="22.22" y1="41.905" x2="22.22" y2="40.64" width="0.6096" layer="1"/>
+<contactref element="U$7" pad="44"/>
+<contactref element="U$7" pad="24"/>
+<wire x1="27.75" y1="31.2" x2="24.13" y2="31.2" width="0.4064" layer="1"/>
+<wire x1="24.13" y1="31.2" x2="24.13" y2="30.48" width="0.4064" layer="1"/>
+<wire x1="37.55" y1="22.2" x2="36.22" y2="22.2" width="0.4064" layer="1"/>
+<wire x1="37.55" y1="22.225" x2="37.55" y2="22.2" width="0.4064" layer="1"/>
 </signal>
 <signal name="E">
@@
 <via x="34.29" y="22.86" extent="1-16" drill="0.6"/>
 <wire x1="34.29" y1="22.86" x2="34.29" y2="24.64" width="0.4064" layer="16"/>
-<wire x1="34.29" y1="24.64" x2="11.51" y2="47.42" width="0.4064" layer="16"/>
+<wire x1="11.51" y1="47.42" x2="34.29" y2="24.64" width="0.4064" layer="16"/>
 </signal>
 <signal name="RX">
 <contactref element="U$7" pad="20"/>
 <contactref element="XB1" pad="2"/>
-<wire x1="34.15" y1="19.6" x2="34.15" y2="21.095" width="0.4064" layer="1"/>
-<wire x1="34.15" y1="21.095" x2="33.655" y2="21.59" width="0.4064" layer="1"/>
-<via x="33.655" y="21.59" extent="1-16" drill="0.6"/>
-<wire x1="33.655" y1="21.59" x2="33.02" y2="22.225" width="0.4064" layer="16"/>
+<wire x1="34.15" y1="19.6" x2="34.15" y2="20.46" width="0.4064" layer="1"/>
+<wire x1="34.15" y1="20.46" x2="33.02" y2="21.59" width="0.4064" layer="1"/>
+<via x="33.02" y="21.59" extent="1-16" drill="0.6"/>
 <wire x1="9.51" y1="47.42" x2="33.02" y2="23.91" width="0.4064" layer="16"/>
-<wire x1="33.02" y1="23.91" x2="33.02" y2="22.225" width="0.4064" layer="16"/>
+<wire x1="33.02" y1="23.91" x2="33.02" y2="21.59" width="0.4064" layer="16"/>
 </signal>
 <signal name="SW8">
@@
 <wire x1="22.225" y1="3.175" x2="22.225" y2="8.255" width="0.4064" layer="1"/>
 <wire x1="22.225" y1="8.255" x2="24.13" y2="10.16" width="0.4064" layer="1"/>
-<wire x1="1.905" y1="8.255" x2="3.81" y2="10.16" width="0.4064" layer="1"/>
 <wire x1="39.37" y1="13.07" x2="39.37" y2="2.54" width="0.4064" layer="1"/>
 <wire x1="39.37" y1="2.54" x2="37.465" y2="0.635" width="0.3048" layer="1"/>
 <wire x1="24.13" y1="1.27" x2="22.225" y2="3.175" width="0.4064" layer="1"/>
-<wire x1="3.175" y1="3.175" x2="22.225" y2="3.175" width="0.4064" layer="1"/>
-<wire x1="1.905" y1="4.445" x2="1.905" y2="8.255" width="0.4064" layer="1"/>
-<wire x1="3.175" y1="3.175" x2="1.905" y2="4.445" width="0.4064" layer="1"/>
+<wire x1="3.81" y1="10.16" x2="24.13" y2="10.16" width="0.4064" layer="16"/>
 </signal>
 <signal name="LED_ENABLE">
