File: Xbee_Remote_32u4/board/remote_smt.sch (EAGLE design)
At the start: 33 parts, among them Q1 MOSFET-NCHANNELSMD, X1 16MHz, X2 USBPTH

Commit message: Fixed up SMT version, added some files zipped.
Parts:
- added JP2, JP3: FIDUCIAL1.5X3, SparkFun:FIDUCIAL1.5X3
- C6, C7: value (none) -> 18pF
Connections:
- net 3.3V: no longer U$7.UVCC
Changed lines of the file:
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@@
 <part name="P+2" library="SparkFun" deviceset="3.3V" device=""/>
 <part name="GND4" library="SparkFun" deviceset="GND" device=""/>
-<part name="C6" library="SparkFun" deviceset="CAP" device="0805"/>
-<part name="C7" library="SparkFun" deviceset="CAP" device="0805"/>
+<part name="C6" library="SparkFun" deviceset="CAP" device="0805" value="18pF"/>
+<part name="C7" library="SparkFun" deviceset="CAP" device="0805" value="18pF"/>
 <part name="GND12" library="SparkFun" deviceset="GND" device=""/>
 <part name="U$11" library="hjohnson_library" deviceset="SPST_SWITCH" device=""/>
@@
 <part name="GND1" library="SparkFun" deviceset="GND" device=""/>
 <part name="GND2" library="SparkFun" deviceset="GND" device=""/>
+<part name="JP2" library="SparkFun" deviceset="FIDUCIAL" device="1.5X3"/>
+<part name="JP3" library="SparkFun" deviceset="FIDUCIAL" device="1.5X3"/>
 </parts>
 <sheets>
@@
 <instance part="FRAME1" gate="G$2" x="147.32" y="0"/>
 <instance part="U$7" gate="G$1" x="129.54" y="121.92" smashed="yes">
-<attribute name="NAME" x="60.96" y="104.14" size="1.778" layer="95"/>
+<attribute name="NAME" x="129.286" y="168.91" size="1.778" layer="95"/>
 <attribute name="VALUE" x="124.46" y="167.64" size="1.778" layer="96"/>
 </instance>
@@
 <instance part="GND1" gate="1" x="121.92" y="53.34"/>
 <instance part="GND2" gate="1" x="233.68" y="134.62"/>
+<instance part="JP2" gate="G$1" x="88.9" y="76.2"/>
+<instance part="JP3" gate="G$1" x="86.36" y="76.2"/>
 </instances>
 <busses>
@@
 </segment>
 <segment>
-<pinref part="U$7" gate="G$1" pin="AVCC1"/>
-<pinref part="U$7" gate="G$1" pin="AVCC"/>
-<pinref part="U$7" gate="G$1" pin="UVCC"/>
 <pinref part="U$7" gate="G$1" pin="VCC1"/>
 <pinref part="U$7" gate="G$1" pin="VCC"/>
 <wire x1="106.68" y1="152.4" x2="106.68" y2="149.86" width="0.1524" layer="91"/>
-<junction x="106.68" y="149.86"/>
-<wire x1="106.68" y1="149.86" x2="106.68" y2="147.32" width="0.1524" layer="91"/>
-<junction x="106.68" y="147.32"/>
-<wire x1="106.68" y1="147.32" x2="106.68" y2="144.78" width="0.1524" layer="91"/>
-<junction x="106.68" y="144.78"/>
-<wire x1="106.68" y1="144.78" x2="106.68" y2="142.24" width="0.1524" layer="91"/>
-<junction x="106.68" y="142.24"/>
 <pinref part="P+1" gate="G$1" pin="3.3V"/>
 <wire x1="106.68" y1="152.4" x2="101.6" y2="152.4" width="0.1524" layer="91"/>
 <junction x="101.6" y="152.4"/>
 <junction x="106.68" y="152.4"/>
-</segment>
-<segment>
+<pinref part="U$7" gate="G$1" pin="AVCC1"/>
+<junction x="106.68" y="142.24"/>
+<pinref part="U$7" gate="G$1" pin="AVCC"/>
+<wire x1="106.68" y1="144.78" x2="106.68" y2="142.24" width="0.1524" layer="91"/>
+<wire x1="106.68" y1="144.78" x2="101.6" y2="144.78" width="0.1524" layer="91"/>
+<wire x1="101.6" y1="144.78" x2="101.6" y2="152.4" width="0.1524" layer="91"/>
+<junction x="106.68" y="144.78"/>
+</segment>
+<segment>
