File: XBee_Receiver/schematic/arduino_card.sch (EAGLE design)
At the start: 22 parts, among them IC1 74LS06N, IC2 74LS06N

Commit message: New revision of remote: Added joystick, shifted parts.
Other:
- note added: "Harry Johnson, https://github.com/hjohnson"
- note removed: "Harry Johnson, hjohnson.posterous.com"
Changed lines of the file:
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@@
 <wire x1="109.22" y1="27.94" x2="109.22" y2="30.48" width="0.4064" layer="94"/>
 <text x="10.16" y="20.32" size="1.778" layer="94">When connecting to XBee, (Arduino TX-&gt;XBee RX) (Arduino RX -&gt; Xbee TX)</text>
-<text x="20.32" y="175.26" size="1.778" layer="97">Harry Johnson, hjohnson.posterous.com</text>
+<text x="20.32" y="175.26" size="1.778" layer="97">Harry Johnson, https://github.com/hjohnson</text>
 <text x="149.86" y="30.48" size="2.54" layer="94">Arduino-Based Rover Control Card</text>
 <text x="12.7" y="162.56" size="1.778" layer="94">Douglas Electronics</text>
